File: thermal-printer-scheme/thermal-printer.sch (KiCad schematic (older format))
At the start: 19 parts, among them U1 L293E

Commit message: corretto il return line per la stampa
Parts:
- removed R? (x5): 1k, symbol R
- added Q? (x2): Q_NPN_BCE, symbol Q_NPN_BCE
- added R? (x3): 1k, symbol R
- added R? (x2): 10k, symbol R
Connections:
- net Enable2 is gone; now on net Enable: R?.1, U1.11 (CE)
- net Earth: now also Q?.3 (E), Q?.3 (E), R?.2
- net Fase1: now also R?.2
- net Fase2: now also R?.2
- net VCC: now also R?.2, R?.2
- net ~Fase1: now also Q?.2 (C), R?.1
- net ~Fase2: now also Q?.2 (C), R?.1
- net Enable1 renamed Enable
- net Enable: now also R?.1
- new net: Q?.1 (B), R?.1 (x2)
Other:
- moved on the sheet: R?
